File: regulator.kicad_sch (KiCad schematic)
At the start: 50 parts, among them J7 39301022, Q1 NX7002BKW, U12 TPS259827ONRGET, U7 LT3045xDD, U8 LT8627SPJV-TRMPBF, U9 TPS7A8500RGRT

Commit message: Finish board, sent out for quote
Parts:
- added C116, C118, C119, C124: 0.1u, Capacitor_SMD:C_0805_2012Metric, symbol Device:C_Small
- added C117, C123: 47u, Capacitor_SMD:C_0805_2012Metric, symbol Device:C_Small
- added C120: 0.01u, Capacitor_SMD:C_0805_2012Metric, symbol Device:C_Small
- added C121, C122, C125: 10u, Capacitor_SMD:C_0805_2012Metric, symbol Device:C_Small
- added L22: LSMGG160808T331RG, My Footprints:IND_LSMG_160808_TAY, symbol My Symbols:LSMGG160808T331RG
- added R147: 12.4K, Resistor_SMD:R_0805_2012Metric, symbol Device:R_Small_US
- added R148: 2.37K, Resistor_SMD:R_0805_2012Metric, symbol Device:R_Small_US
- added R149, R150, R151, R152: 10k, Resistor_SMD:R_0603_1608Metric, symbol Device:R_Small_US
- added U25: TPS7A8500RGRT, My Footprints:QFN50P350X350X100-21N, symbol My Symbols:TPS7A8500RGRT
- added U26: ADS1115IDGSR, My Footprints:SOP50P490X110-10N, symbol My Symbols:ADS1115IDGSR
Connections:
- net +3.3V: now also R151.1
- net +6.0V: now also U8.30 (PVIN), C116.1, L22.2, R149.1
- net GND: now also C116.2, C117.2, C118.2, C119.2, C121.2, C122.2, C123.2, C124.2, C125.2, R148.2, R150.2, R152.2, U25.18 (GND), U25.21 (GND_TH), U25.8 (GND), U26.1 (ADDR), U26.3 (GND), U26.7 (AIN3); no longer U8.29 (GND), U8.30 (GND), U8.31 (GND), U8.32 (GND)
- net sw: now also U8.29 (SW)
- net Imon: now reaches R122.1, U12.9 (IMON)
- net Imon: now also U26.4 (AIN0)
- new net: R149.2, R150.1, U26.5 (AIN1)
- new net: C118.1, U25.13 (NR/SS)
- new net: R151.2, R152.1, U26.6 (AIN2)
- new net: C120.2, R147.2, R148.1, U25.3 (FB)
- new net +5VD: C120.1, C121.1, C122.1, C123.1, C124.1, C125.1, R147.1, U25.1 (OUT), U25.19 (OUT), U25.20 (OUT), U26.8 (VDD)
- new net +6v_U25: C117.1, C119.1, L22.1, U25.14 (EN), U25.15 (IN), U25.16 (IN), U25.17 (IN)
- new net I2C.SCL: U26.10 (SCL)
- new net I2C.SDA: U26.9 (SDA)
Other:
- moved on the sheet: C44, C47, C55, C57, C58, C61, C65, C72, C74, C75, C77, C78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
